File: UHBadge.kicad_pcb (KiCad board)
At the start: 2 copper layers, 70 x 117.6 mm, 103 parts, among them J1 Conn_01x03_MountingPin, J3 LEMO2, J4 Micro_SD_Card, J5 Conn_01x08_MountingPin, P1 USB_C_Plug_USB2.0, Q1 Si1308EDL, SW1 Boot, SW2 Run, SW3 Up, SW4 Down, SW5 Left, SW6 Right, U1 RP2350A, U2 MCP73871, U3 W25Q128JVS, U4 SRV05-4, U5 Conn, U6 ST25DV64K-JFR6D3, U7 Radio Module 2, Y1 ABM8-272-T3

Commit message: Finished the connections. Made some graphics.
Parts:
- added G***: LOGO, LOGO, B.Cu at (175.2, 60.9)
- added G***: LOGO, LOGO, B.Cu at (135.0, 52.5)
- added G***: LOGO, LOGO, B.Cu at (115.2, 60.9)
- added G***: LOGO, LOGO, B.Cu at (135.2, 60.9)
- added G***: LOGO, LOGO, B.Cu at (155.2, 60.9)
- added G***: LOGO, LOGO, B.Cu at (101.2, 60.4)
- moved G*** 0.40 mm to (165.4, 105.0)
- moved C11 0.37 mm to (128.4, 97.8)
- moved C4 0.30 mm to (131.2, 96.4)
- moved R4 0.29 mm to (159.8, 101.2)
- moved C17 0.25 mm to (117.7, 125.0)
Routing:
- net SD-DAT0: track 0.00 -> 62.3 mm, vias 0 -> 4
- net SD-DAT1: track 0.00 -> 61.6 mm, vias 0 -> 4
- net SD-DAT2: track 0.00 -> 53.9 mm, vias 0 -> 4
- net SD-DAT3: track 0.00 -> 52.5 mm, vias 0 -> 4
- net -BATT: track 456.6 -> 445.6 mm, vias 77 -> 76
- net RUN: track 64.6 -> 60.4 mm
- net USB_C_VBUS: track 97.1 -> 101.0 mm, vias 7 -> 6
- net E-INK_CS: track 51.0 -> 53.1 mm
- net E-INK_SCL: track 49.6 -> 51.1 mm
- net E-INK_SDA: track 47.7 -> 49.0 mm
- net GPIO24: track 33.3 -> 34.5 mm
- net SWCLK: track 60.7 -> 61.3 mm
- net E-INK_BUSY: track 71.3 -> 70.7 mm
- net GPIO23: track 20.7 -> 21.3 mm

Commit message: Finished the design.
Parts:
- removed the G*** at (120.8, 139.4)
- removed the G*** at (116.2, 139.4)
- removed the G*** at (130.2, 58.5)
- removed the G*** at (139.8, 58.6)
- added G***: LOGO, LOGO, F.Cu at (140.8, 58.5)
- added G***: LOGO, LOGO, F.Cu at (129.2, 58.5)
- added G***: LOGO, LOGO, F.Cu at (161.4, 72.4)
Other:
- board text added: "Powered by GitHub API"
- board text added: "Powered by RP2350"
- board text removed: "GPIO4"
- board text removed: "GPIO5"
