File: UHBadge.kicad_sch (KiCad schematic)
At the start: 82 parts, among them J1 Conn_01x03_MountingPin, J2 Conn_01x10_MountingPin, P1 USB_C_Plug_USB2.0, Q1 Si1308EDL, SW1 Boot, SW2 Run, SW3 Up, SW4 Down, SW5 Left, SW6 Right, U1 RP2350A, U2 MCP73871, U3 W25Q128JVS, U4 SRV05-4, U5 Conn, U6 ST25DV64K-JFR6D3, Y1 ABM8-272-T3

Commit message: Added the e-ink display. Made the button design.
Parts:
- SW1, SW2, SW3, SW4, SW5, SW6: footprint Button_Switch_THT:SW_PUSH_6mm -> Button_Switch_SMD:SW_SPST_EVQP2_MiddlePushTravel_H2.5mm
Changed lines of the file:
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@@
 	(title_block
 		(title "Universal Hacker Badge")
-		(date "2026-08-27")
+		(date "2026-08-28")
 		(rev "1.0.0")
 		(company "Gianluca Rainis")
@@
 			)
 		)
-		(property "Footprint" "Button_Switch_THT:SW_PUSH_6mm"
+		(property "Footprint" "Button_Switch_SMD:SW_SPST_EVQP2_MiddlePushTravel_H2.5mm"
 			(at 172.72 240.03 0)
 			(hide yes)
@@
 			)
 		)
-		(property "Footprint" "Button_Switch_THT:SW_PUSH_6mm"
+		(property "Footprint" "Button_Switch_SMD:SW_SPST_EVQP2_MiddlePushTravel_H2.5mm"
 			(at 217.17 185.42 0)
 			(hide yes)
@@
 			)
 		)
-		(property "Footprint" "Button_Switch_THT:SW_PUSH_6mm"
+		(property "Footprint" "Button_Switch_SMD:SW_SPST_EVQP2_MiddlePushTravel_H2.5mm"
 			(at 217.17 173.99 0)
 			(hide yes)
@@
 			)
 		)
-		(property "Footprint" "Button_Switch_THT:SW_PUSH_6mm"
+		(property "Footprint" "Button_Switch_SMD:SW_SPST_EVQP2_MiddlePushTravel_H2.5mm"
 			(at 217.17 208.28 0)
 			(hide yes)
@@
 			)
 		)
-		(property "Footprint" "Button_Switch_THT:SW_PUSH_6mm"
+		(property "Footprint" "Button_Switch_SMD:SW_SPST_EVQP2_MiddlePushTravel_H2.5mm"
 			(at 217.17 196.85 0)
 			(hide yes)
@@
 			)
 		)
-		(property "Footprint" "Button_Switch_THT:SW_PUSH_6mm"
+		(property "Footprint" "Button_Switch_SMD:SW_SPST_EVQP2_MiddlePushTravel_H2.5mm"
 			(at 205.74 232.41 0)
 			(hide yes)

Commit message: Connected the support components to the e-ink display. Placed the RP2350 and started connecting the support components.
Parts:
- removed C14, C15: 100nF, Capacitor_SMD:C_0402_1005Metric, symbol Device:C
- C5: value 4.7uF -> 100nF
- J1: footprint Connector_PinHeader_1.00mm:PinHeader_1x03_P1.00mm_Vertical -> Connector_PinHeader_2.54mm:PinHeader_1x03_P2.54mm_Vertical
- J2: footprint Connector_PinHeader_1.00mm:PinHeader_1x10_P1.00mm_Vertical -> Connector_PinHeader_2.54mm:PinHeader_1x10_P2.54mm_Vertical
Other:
- moved on the sheet: C1, C2, C3, C4, C5, C6, J2, P1, R1, R4

Commit message: RP2350 Support components placement, USB-C connection and NFC component placement.
Other:
- moved on the sheet: C10, C11, C12, C13, C4, C5, C6, C7, C8, C9, R11, R9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

Commit message: Battery Port Placement. Finished the recharge system. Placed the mounting holes. Started filling the areas and connecting the components.
Parts:
- removed BT1: Battery, symbol Device:Battery
- added J3: LEMO2, Connector_Molex:Molex_CLIK-Mate_502494-0270_1x02-1MP_P2.00mm_Horizontal, symbol Connector:LEMO2
Connections:
- net +3V3: now also J3.1
- net -BATT: now also R9.2, J3.2; no longer SW1.1
- net QSPI_SS: now also SW1.1; no longer R9.2
Other:
- moved on the sheet: C10, C11, C12, C13, C4, C5, C6, C7, C8, C9, J1, R11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

Commit message: Added two new mounting holes. Fixed the NFC footprint. Started working on the design.
Parts:
- added H3, H4: MountingHole_Pad, MountingHole:MountingHole_2.2mm_M2_Pad_Via, symbol Mechanical:MountingHole_Pad
Connections:
- net -BATT: now also H3.1, H4.1

Commit message: Added the Pi Radio Module 2.
Parts:
- added R18: 470Ω, Resistor_SMD:R_0402_1005Metric, symbol Device:R
- added R19: 10kΩ, Resistor_SMD:R_0402_1005Metric, symbol Device:R
- added U7: Radio Module 2, CustomFootprints:rpi_rmc20452t, symbol RPI_WIFI:RPI_RMC20452T
Connections:
- net +3V3: now also U7.14 (VDDIO), U7.16 (VIN)
- net -BATT: now also U7.1 (GND), U7.11 (GND), U7.15 (GND), U7.21 (GND), U7.4 (GND), U7.7 (GND)
- net GPIO23: now reaches U1.35 (GPIO23)
- net GPIO23: now also U7.12 (WL_ON), U7.13 (BT_ON)
- net GPIO24: now reaches U1.36 (GPIO24)
- net GPIO24: now also R18.2, R19.2, U7.5 (DI)
- net GPIO25: now reaches U1.37 (GPIO25)
- net GPIO25: now also U7.9 (CS)
- net GPIO29: now reaches U1.43 (GPIO29/ADC3)
- net GPIO29: now also U7.3 (SCLK)
- new net: R19.1, U7.10 (nIRQ)
- new net: R18.1, U7.6 (DO)
- no-connect marks 4 -> 7
Other:
- note added: "RPI Radio Module 2"

Commit message: Added the microSD card slot. Moved the SW pins. Removed two expansion pins. Added some graphical designs.
Parts:
- removed J2: Conn_01x10_MountingPin, Connector_PinHeader_2.54mm:PinHeader_1x10_P2.54mm_Vertical, symbol Connector_Generic_MountingPin:Conn_01x10_MountingPin
- added C36: 10uF, Capacitor_SMD:C_0402_1005Metric, symbol Device:C
- added J4: Micro_SD_Card, Connector_Card:microSD_HC_Hirose_DM3AT-SF-PEJM5, symbol Connector:Micro_SD_Card
- added J5: Conn_01x08_MountingPin, Connector_PinHeader_2.54mm:PinHeader_1x08_P2.54mm_Vertical, symbol Connector_Generic_MountingPin:Conn_01x08_MountingPin
Connections:
- net +3V3: now also C36.1, J4.4 (VDD), J5.1 (Pin_1)
- net -BATT: now also C36.2, J4.6 (VSS), J4.SH (SHIELD), J5.8 (Pin_8), J5.MP (MountPin)
- net ADC0: now also J5.6 (Pin_6)
- net ADC1: now also J5.7 (Pin_7)
- net GPIO0: now also J5.2 (Pin_2)
- net GPIO1: now also J5.3 (Pin_3)
- net GPIO2: now also J5.4 (Pin_4)
- net GPIO3: now also J5.5 (Pin_5)
- net SD-DAT0: now reaches U1.31 (GPIO19)
- net SD-DAT0: now also J4.7 (DAT0)
- net SD-DAT1: now reaches U1.32 (GPIO20)
- net SD-DAT1: now also J4.8 (DAT1)
- net SD-DAT2: now reaches U1.33 (GPIO21)
- net SD-DAT2: now also J4.1 (DAT2)
- net SD-DAT3: now reaches U1.34 (GPIO22)
- net SD-DAT3: now also J4.2 (DAT3/CD)
- net GPIO4 renamed SD-CLK
- net SD-CLK: now also J4.5 (CLK)
- net GPIO5 renamed SD-CMD
- net SD-CMD: now also J4.3 (CMD)
Other:
- note added: "Micro SD"
- moved on the sheet: C20, C21, R10, U4, Y1

Commit message: Added confirm button. Moved the NFC tag. Fixed the design.
Parts:
- removed J1: Conn_01x03_MountingPin, Connector_PinHeader_2.54mm:PinHeader_1x03_P2.54mm_Vertical, symbol Connector_Generic_MountingPin:Conn_01x03_MountingPin
- removed J5: Conn_01x08_MountingPin, Connector_PinHeader_2.54mm:PinHeader_1x08_P2.54mm_Vertical, symbol Connector_Generic_MountingPin:Conn_01x08_MountingPin
- added SW7: Confirm, Button_Switch_SMD:SW_SPST_EVQP2_MiddlePushTravel_H2.5mm, symbol Switch:SW_Push
- added TP1, TP10, TP11, TP2, TP3, TP4, TP5, TP6, TP7, TP8, TP9: TestPoint, TestPoint:TestPoint_Pad_D1.0mm, symbol Connector:TestPoint
Connections:
- net +3V3: now also TP4.1
- net -BATT: now also SW7.2, TP11.1, TP2.1
- net ADC0: now also TP9.1
- net ADC1: now also TP10.1
- net GPIO0: now also TP5.1
- net GPIO1: now also TP6.1
- net GPIO2: now also TP7.1
- net GPIO3: now also TP8.1
- net SWCLK: now also TP1.1
- net SWDIO: now also TP3.1
- net CONFIRM: now reaches U1.42 (GPIO28/ADC2)
- net CONFIRM: now also SW7.1
Other:
- note added: "RP2350"
- moved on the sheet: C1, C2, C3, L1, R1, R2, R3, SW3, SW4, SW5, SW6, U1
